File: PCB/power.kicad_sch (KiCad schematic)
At the start: 45 parts, among them Q1 AO3401A, U5 LM317_SOT-223, U6 LM317_SOT-223, U7 TPS65131RGE, U8 LM317_SOT-223, U9 LM337_SOT223

Commit message: Added filter capacitors to OPA1622 circuitry
Parts:
- C21, C23, C24, C30, C50, C51: JLCPCBPn C15849 -> (none); LCSC Part # (none) -> C15849
- C22, C29, C41, C48, C49: JLCPCBPn C1525 -> (none); LCSC Part # (none) -> C1525
- C37, C40: JLCPCBPn C19666 -> (none); LCSC Part # (none) -> C19666
- C38: JLCPCBPn C88896 -> (none); LCSC Part # (none) -> C88896
- C39, C46, C47: JLCPCBPn C84419 -> (none); LCSC Part # (none) -> C84419
- C42: JLCPCBPn C16772 -> (none); LCSC Part # (none) -> C16772
- C43: JLCPCBPn C88938 -> (none); LCSC Part # (none) -> C88938
- C44: JLCPCBPn C15195 -> (none); LCSC Part # (none) -> C15195
- C45: JLCPCBPn C1538 -> (none); LCSC Part # (none) -> C1538
- D1, D2: JLCPCBPn C82461 -> (none); LCSC Part # (none) -> C82461
- L1, L2: JLCPCBPn C6707914 -> (none); LCSC Part # (none) -> C6707914
- Q1: JLCPCBPn C15127 -> (none); LCSC Part # (none) -> C15127
- R43, R53: JLCPCBPn C274891 -> (none); LCSC Part # (none) -> C274891
- R44, R54, R62, R63: JLCPCBPn C25094 -> (none); LCSC Part # (none) -> C25094
- R55, R59: JLCPCBPn C26083 -> (none); LCSC Part # (none) -> C26083
- R56: JLCPCBPn C185459 -> (none); LCSC Part # (none) -> C185459
- R57: JLCPCBPn C25076 -> (none); LCSC Part # (none) -> C25076
- R58: JLCPCBPn C25755 -> (none); LCSC Part # (none) -> C25755
- R60, R61: JLCPCBPn C416571 -> (none); LCSC Part # (none) -> C416571
- U5, U6, U8: JLCPCBPn C84244 -> (none); LCSC Part # (none) -> C84244
- U7: JLCPCBPn C87663 -> (none); LCSC Part # (none) -> C87663
- U9: JLCPCBPn C527400 -> (none); LCSC Part # (none) -> C527400
Changed lines of the file:
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@@
 			)
 		)
-		(property "JLCPCBPn" "C15849"
+		(property "LCSC Part #" "C15849"
 			(at 255.27 72.39 0)
 			(effects
@@
 			)
 		)
-		(property "JLCPCBPn" "C1525"
+		(property "LCSC Part #" "C1525"
 			(at 204.47 76.2 0)
 			(effects
@@
 			)
 		)
-		(property "JLCPCBPn" "C88896"
+		(property "LCSC Part #" "C88896"
 			(at 170.18 38.1 0)
 			(effects
@@
 			)
 		)
-		(property "JLCPCBPn" "C1538"
+		(property "LCSC Part #" "C1538"
 			(at 124.46 80.01 0)
 			(effects
@@
 			)
 		)
-		(property "JLCPCBPn" "C185459"
+		(property "LCSC Part #" "C185459"
 			(at 160.02 48.26 0)
 			(effects
@@
 			)
 		)
-		(property "JLCPCBPn" "C416571"
+		(property "LCSC Part #" "C416571"
 			(at 224.79 54.61 0)
 			(effects
@@
 			)
 		)
-		(property "JLCPCBPn" "C15127"
+		(property "LCSC Part #" "C15127"
 			(at 54.61 35.56 0)
 			(effects
@@
 			)
 		)
-		(property "JLCPCBPn" "C25094"
+		(property "LCSC Part #" "C25094"
 			(at 90.17 163.83 0)
 			(effects
@@
 			)
 		)
-		(property "JLCPCBPn" "C1525"
+		(property "LCSC Part #" "C1525"
 			(at 55.88 163.83 0)
 			(effects
@@
 			)
 		)
-		(property "JLCPCBPn" "C84419"
+		(property "LCSC Part #" "C84419"
 			(at 185.42 38.1 0)
 			(effects
@@
 			)
 		)
-		(property "JLCPCBPn" "C88938"
+		(property "LCSC Part #" "C88938"
 			(at 143.51 63.5 0)
 			(effects
@@
 			)
 		)
-		(property "JLCPCBPn" "C25094"
+		(property "LCSC Part #" "C25094"
 			(at 90.17 118.11 0)
 			(effects
@@
 			)
 		)
-		(property "JLCPCBPn" "C84419"
+		(property "LCSC Part #" "C84419"
 			(at 191.77 76.2 0)
 			(effects
@@
 			)
 		)
-		(property "JLCPCBPn" "C15849"
+		(property "LCSC Part #" "C15849"
 			(at 104.14 163.83 0)
 			(effects
@@
 			)
 		)
-		(property "JLCPCBPn" "C6707914"
+		(property "LCSC Part #" "C6707914"
 			(at 156.21 76.2 0)
 			(effects
@@
 			)
 		)
-		(property "JLCPCBPn" "C84244"
+		(property "LCSC Part #" "C84244"
 			(at 73.66 158.75 0)
 			(effects
@@
 			)
 		)
-		(property "JLCPCBPn" "C15849"
+		(property "LCSC Part #" "C15849"
 			(at 40.64 118.11 0)
 			(effects
@@
 			)
 		)
-		(property "JLCPCBPn" "C84244"
+		(property "LCSC Part #" "C84244"
 			(at 224.79 33.02 0)
 			(effects
@@
 			)
 		)
-		(property "JLCPCBPn" "C26083"
+		(property "LCSC Part #" "C26083"
 			(at 133.35 63.5 0)
 			(effects
@@
 			)
 		)
-		(property "JLCPCBPn" "C82461"
+		(property "LCSC Part #" "C82461"
 			(at 105.41 33.02 0)
 			(effects
@@
 			)
 		)
-		(property "JLCPCBPn" "C1525"
+		(property "LCSC Part #" "C1525"
 			(at 60.96 67.31 0)
 			(effects
@@
 			)
 		)
-		(property "JLCPCBPn" "C19666"
+		(property "LCSC Part #" "C19666"
 			(at 68.58 36.83 0)
 			(effects
@@
 			)
 		)
-		(property "JLCPCBPn" "C274891"
+		(property "LCSC Part #" "C274891"
 			(at 73.66 172.72 0)
 			(effects
@@
 			)
 		)
-		(property "JLCPCBPn" "C15849"
+		(property "LCSC Part #" "C15849"
 			(at 40.64 163.83 0)
 			(effects
@@
 			)
 		)
-		(property "JLCPCBPn" "C87663"
+		(property "LCSC Part #" "C87663"
 			(at 101.6 62.23 0)
 			(effects
@@
 			)
 		)
-		(property "JLCPCBPn" "C19666"
+		(property "LCSC Part #" "C19666"
 			(at 40.64 67.31 0)
 			(effects
@@
 			)
 		)
-		(property "JLCPCBPn" "C16772"
+		(property "LCSC Part #" "C16772"
 			(at 144.78 52.07 0)
 			(effects
@@
 			)
 		)
-		(property "JLCPCBPn" "C25076"
+		(property "LCSC Part #" "C25076"
 			(at 49.53 59.69 0)
 			(effects
@@
 			)
 		)
-		(property "JLCPCBPn" "C25094"
+		(property "LCSC Part #" "C25094"
 			(at 241.3 63.5 0)
 			(effects
@@
 			)
 		)
-		(property "JLCPCBPn" "C527400"
+		(property "LCSC Part #" "C527400"
 			(at 224.79 67.31 0)
 			(effects
@@
 			)
 		)
-		(property "JLCPCBPn" "C26083"
+		(property "LCSC Part #" "C26083"
 			(at 160.02 38.1 0)
 			(effects
@@
 			)
 		)
-		(property "JLCPCBPn" "C84244"
+		(property "LCSC Part #" "C84244"
 			(at 73.66 113.03 0)
 			(effects
@@
 			)
 		)
-		(property "JLCPCBPn" "C274891"
+		(property "LCSC Part #" "C274891"
 			(at 73.66 127 0)
 			(effects
@@
 			)
 		)
-		(property "JLCPCBPn" "C82461"
+		(property "LCSC Part #" "C82461"
 			(at 175.26 74.93 0)
 			(effects
@@
 			)
 		)
-		(property "JLCPCBPn" "C6707914"
+		(property "LCSC Part #" "C6707914"
 			(at 85.09 33.02 0)
 			(effects
@@
 			)
 		)
-		(property "JLCPCBPn" "C1525"
+		(property "LCSC Part #" "C1525"
 			(at 200.66 38.1 0)
 			(effects
@@
 			)
 		)
-		(property "JLCPCBPn" "C15195"
+		(property "LCSC Part #" "C15195"
 			(at 118.11 80.01 0)
 			(effects
@@
 			)
 		)
-		(property "JLCPCBPn" "C1525"
+		(property "LCSC Part #" "C1525"
 			(at 55.88 118.11 0)
 			(effects
@@
 			)
 		)
-		(property "JLCPCBPn" "C25755"
+		(property "LCSC Part #" "C25755"
 			(at 133.35 55.88 0)
 			(effects
@@
 			)
 		)
-		(property "JLCPCBPn" "C84419"
+		(property "LCSC Part #" "C84419"
 			(at 185.42 76.2 0)
 			(effects
@@
 			)
 		)
-		(property "JLCPCBPn" "C416571"
+		(property "LCSC Part #" "C416571"
 			(at 224.79 45.72 0)
 			(effects
@@
 			)
 		)
-		(property "JLCPCBPn" "C25094"
+		(property "LCSC Part #" "C25094"
 			(at 241.3 36.83 0)
 			(effects
@@
 			)
 		)
-		(property "JLCPCBPn" "C15849"
+		(property "LCSC Part #" "C15849"
 			(at 104.14 118.11 0)
 			(effects
@@
 			)
 		)
-		(property "JLCPCBPn" "C15849"
+		(property "LCSC Part #" "C15849"
 			(at 256.54 38.1 0)
 			(effects

Commit message: Changed the BOM field for JLCPCB to the original name instead of LCSC
Parts:
- C21, C23, C24, C30, C50, C51: JLCPCB Part # (none) -> C15849; LCSC Part # C15849 -> (none)
- C22, C29, C41, C48, C49: JLCPCB Part # (none) -> C1525; LCSC Part # C1525 -> (none)
- C37, C40: JLCPCB Part # (none) -> C19666; LCSC Part # C19666 -> (none)
- C38: JLCPCB Part # (none) -> C88896; LCSC Part # C88896 -> (none)
- C39, C46, C47: JLCPCB Part # (none) -> C84419; LCSC Part # C84419 -> (none)
- C42: JLCPCB Part # (none) -> C16772; LCSC Part # C16772 -> (none)
- C43: JLCPCB Part # (none) -> C88938; LCSC Part # C88938 -> (none)
- C44: JLCPCB Part # (none) -> C15195; LCSC Part # C15195 -> (none)
- C45: JLCPCB Part # (none) -> C1538; LCSC Part # C1538 -> (none)
- D1, D2: JLCPCB Part # (none) -> C82461; LCSC Part # C82461 -> (none)
- L1, L2: JLCPCB Part # (none) -> C6707914; LCSC Part # C6707914 -> (none)
- Q1: JLCPCB Part # (none) -> C15127; LCSC Part # C15127 -> (none)
- R43, R53: JLCPCB Part # (none) -> C274891; LCSC Part # C274891 -> (none)
- R44, R54, R62, R63: JLCPCB Part # (none) -> C25094; LCSC Part # C25094 -> (none)
- R55, R59: JLCPCB Part # (none) -> C26083; LCSC Part # C26083 -> (none)
- R56: JLCPCB Part # (none) -> C185459; LCSC Part # C185459 -> (none)
- R57: JLCPCB Part # (none) -> C25076; LCSC Part # C25076 -> (none)
- R58: JLCPCB Part # (none) -> C25755; LCSC Part # C25755 -> (none)
- R60, R61: JLCPCB Part # (none) -> C416571; LCSC Part # C416571 -> (none)
- U5, U6, U8: JLCPCB Part # (none) -> C84244; LCSC Part # C84244 -> (none)
- U7: JLCPCB Part # (none) -> C87663; LCSC Part # C87663 -> (none)
- U9: JLCPCB Part # (none) -> C527400; LCSC Part # C527400 -> (none)
Changed lines of the file:
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@@
 			)
 		)
-		(property "LCSC Part #" "C15849"
+		(property "JLCPCB Part #" "C15849"
 			(at 255.27 72.39 0)
 			(effects
@@
 			)
 		)
-		(property "LCSC Part #" "C1525"
+		(property "JLCPCB Part #" "C1525"
 			(at 204.47 76.2 0)
 			(effects
@@
 			)
 		)
-		(property "LCSC Part #" "C88896"
+		(property "JLCPCB Part #" "C88896"
 			(at 170.18 38.1 0)
 			(effects
@@
 			)
 		)
-		(property "LCSC Part #" "C1538"
+		(property "JLCPCB Part #" "C1538"
 			(at 124.46 80.01 0)
 			(effects
@@
 			)
 		)
-		(property "LCSC Part #" "C185459"
+		(property "JLCPCB Part #" "C185459"
 			(at 160.02 48.26 0)
 			(effects
@@
 			)
 		)
-		(property "LCSC Part #" "C416571"
+		(property "JLCPCB Part #" "C416571"
 			(at 224.79 54.61 0)
 			(effects
@@
 			)
 		)
-		(property "LCSC Part #" "C15127"
+		(property "JLCPCB Part #" "C15127"
 			(at 54.61 35.56 0)
 			(effects
@@
 			)
 		)
-		(property "LCSC Part #" "C25094"
+		(property "JLCPCB Part #" "C25094"
 			(at 90.17 163.83 0)
 			(effects
@@
 			)
 		)
-		(property "LCSC Part #" "C1525"
+		(property "JLCPCB Part #" "C1525"
 			(at 55.88 163.83 0)
 			(effects
@@
 			)
 		)
-		(property "LCSC Part #" "C84419"
+		(property "JLCPCB Part #" "C84419"
 			(at 185.42 38.1 0)
 			(effects
@@
 			)
 		)
-		(property "LCSC Part #" "C88938"
+		(property "JLCPCB Part #" "C88938"
 			(at 143.51 63.5 0)
 			(effects
@@
 			)
 		)
-		(property "LCSC Part #" "C25094"
+		(property "JLCPCB Part #" "C25094"
 			(at 90.17 118.11 0)
 			(effects
@@
 			)
 		)
-		(property "LCSC Part #" "C84419"
+		(property "JLCPCB Part #" "C84419"
 			(at 191.77 76.2 0)
 			(effects
@@
 			)
 		)
-		(property "LCSC Part #" "C15849"
+		(property "JLCPCB Part #" "C15849"
 			(at 104.14 163.83 0)
 			(effects
@@
 			)
 		)
-		(property "LCSC Part #" "C6707914"
+		(property "JLCPCB Part #" "C6707914"
 			(at 156.21 76.2 0)
 			(effects
@@
 			)
 		)
-		(property "LCSC Part #" "C84244"
+		(property "JLCPCB Part #" "C84244"
 			(at 73.66 158.75 0)
 			(effects
@@
 			)
 		)
-		(property "LCSC Part #" "C15849"
+		(property "JLCPCB Part #" "C15849"
 			(at 40.64 118.11 0)
 			(effects
@@
 			)
 		)
-		(property "LCSC Part #" "C84244"
+		(property "JLCPCB Part #" "C84244"
 			(at 224.79 33.02 0)
 			(effects
@@
 			)
 		)
-		(property "LCSC Part #" "C26083"
+		(property "JLCPCB Part #" "C26083"
 			(at 133.35 63.5 0)
 			(effects
@@
 			)
 		)
-		(property "LCSC Part #" "C82461"
+		(property "JLCPCB Part #" "C82461"
 			(at 105.41 33.02 0)
 			(effects
@@
 			)
 		)
-		(property "LCSC Part #" "C1525"
+		(property "JLCPCB Part #" "C1525"
 			(at 60.96 67.31 0)
 			(effects
@@
 			)
 		)
-		(property "LCSC Part #" "C19666"
+		(property "JLCPCB Part #" "C19666"
 			(at 68.58 36.83 0)
 			(effects
@@
 			)
 		)
-		(property "LCSC Part #" "C274891"
+		(property "JLCPCB Part #" "C274891"
 			(at 73.66 172.72 0)
 			(effects
@@
 			)
 		)
-		(property "LCSC Part #" "C15849"
+		(property "JLCPCB Part #" "C15849"
 			(at 40.64 163.83 0)
 			(effects
@@
 			)
 		)
-		(property "LCSC Part #" "C87663"
+		(property "JLCPCB Part #" "C87663"
 			(at 101.6 62.23 0)
 			(effects
@@
 			)
 		)
-		(property "LCSC Part #" "C19666"
+		(property "JLCPCB Part #" "C19666"
 			(at 40.64 67.31 0)
 			(effects
@@
 			)
 		)
-		(property "LCSC Part #" "C16772"
+		(property "JLCPCB Part #" "C16772"
 			(at 144.78 52.07 0)
 			(effects
@@
 			)
 		)
-		(property "LCSC Part #" "C25076"
+		(property "JLCPCB Part #" "C25076"
 			(at 49.53 59.69 0)
 			(effects
@@
 			)
 		)
-		(property "LCSC Part #" "C25094"
+		(property "JLCPCB Part #" "C25094"
 			(at 241.3 63.5 0)
 			(effects
@@
 			)
 		)
-		(property "LCSC Part #" "C527400"
+		(property "JLCPCB Part #" "C527400"
 			(at 224.79 67.31 0)
 			(effects
@@
 			)
 		)
-		(property "LCSC Part #" "C26083"
+		(property "JLCPCB Part #" "C26083"
 			(at 160.02 38.1 0)
 			(effects
@@
 			)
 		)
-		(property "LCSC Part #" "C84244"
+		(property "JLCPCB Part #" "C84244"
 			(at 73.66 113.03 0)
 			(effects
@@
 			)
 		)
-		(property "LCSC Part #" "C274891"
+		(property "JLCPCB Part #" "C274891"
 			(at 73.66 127 0)
 			(effects
@@
 			)
 		)
-		(property "LCSC Part #" "C82461"
+		(property "JLCPCB Part #" "C82461"
 			(at 175.26 74.93 0)
 			(effects
@@
 			)
 		)
-		(property "LCSC Part #" "C6707914"
+		(property "JLCPCB Part #" "C6707914"
 			(at 85.09 33.02 0)
 			(effects
@@
 			)
 		)
-		(property "LCSC Part #" "C1525"
+		(property "JLCPCB Part #" "C1525"
 			(at 200.66 38.1 0)
 			(effects
@@
 			)
 		)
-		(property "LCSC Part #" "C15195"
+		(property "JLCPCB Part #" "C15195"
 			(at 118.11 80.01 0)
 			(effects
@@
 			)
 		)
-		(property "LCSC Part #" "C1525"
+		(property "JLCPCB Part #" "C1525"
 			(at 55.88 118.11 0)
 			(effects
@@
 			)
 		)
-		(property "LCSC Part #" "C25755"
+		(property "JLCPCB Part #" "C25755"
 			(at 133.35 55.88 0)
 			(effects
@@
 			)
 		)
-		(property "LCSC Part #" "C84419"
+		(property "JLCPCB Part #" "C84419"
 			(at 185.42 76.2 0)
 			(effects
@@
 			)
 		)
-		(property "LCSC Part #" "C416571"
+		(property "JLCPCB Part #" "C416571"
 			(at 224.79 45.72 0)
 			(effects
@@
 			)
 		)
-		(property "LCSC Part #" "C25094"
+		(property "JLCPCB Part #" "C25094"
 			(at 241.3 36.83 0)
 			(effects
@@
 			)
 		)
-		(property "LCSC Part #" "C15849"
+		(property "JLCPCB Part #" "C15849"
 			(at 104.14 118.11 0)
 			(effects
@@
 			)
 		)
-		(property "LCSC Part #" "C15849"
+		(property "JLCPCB Part #" "C15849"
 			(at 256.54 38.1 0)
 			(effects
